File: rj45-mapper.kicad_pcb (KiCad board)
At the start: 2 copper layers, 75 x 50 mm, 34 parts, among them J1 RC01937, J2 USB-C_5V, Q1 MMBT3904, U1 ULN2803A

Commit message: Rev A2: right-angle jack on the 8P8C drawing, plug-path check
The RC01937 is a top-entry jack, so the case wall faced a closed side. J1 is now
an unshielded right-angle jack on the TE 5555164 / Amphenol 54602 land pattern
(0.89 mm pins, 3.25 mm pegs), bought separately, with its plug face flush with
the board edge; the TE model is aligned to the pads and the face. The shield
channel is gone. fit_check.py now casts rays along the plug path from outside
the case into the jack.
Parts:
- removed D10: RED, LED_SMD:LED_1206_3216Metric
- removed Q1: MMBT3904, Package_TO_SOT_SMD:SOT-23
- removed R13: 2.7k, Resistor_SMD:R_0805_2012Metric
- removed R14: 10k, Resistor_SMD:R_0805_2012Metric
- removed R15: 330, Resistor_SMD:R_0805_2012Metric
- J1: value RC01937 -> TE 5555164-1 or equal, RA unshielded; footprint rj45-mapper:RJ45_RCH_RC01937 -> rj45-mapper:RJ45_8P8C_RightAngle
- moved J1 1.22 mm to (124.4, 114.2)
Routing:
- net /OS: track 56.3 -> 0.00 mm, vias 2 -> 0
- net /SHLD: track 18.9 -> 0.00 mm
- net /5V: track 142.5 -> 136.5 mm
- net /QB: track 4.97 -> 0.00 mm
- net /GND: track 13.6 -> 10.3 mm, vias 47 -> 46
- net /LEDAS: track 3.09 -> 0.00 mm
- net /IN8: track 6.81 -> 5.59 mm
- net /IN6: track 6.81 -> 5.59 mm
- net /IN4: track 6.81 -> 5.59 mm
- net /IN2: track 6.81 -> 5.59 mm
- net /IN7: track 9.35 -> 8.13 mm
- net /IN5: track 9.35 -> 8.13 mm
- net /IN3: track 9.35 -> 8.13 mm
- net /IN1: track 9.35 -> 8.13 mm
Other:
- board text added: "RJ45 MAPPER rev A2"
- board text added: "Rix rev A2 2026-10-22"
- board text removed: "RJ45 MAPPER rev A"
- board text removed: "Rix rev A 2026-10-22"
- board text removed: "S"
